File: arduino_uno_grbl_shield.sch (KiCad schematic (older format))
At the start: 21 parts

Commit message: Schema v0.1
Parts:
- removed U? (x7): TLP185, MFSOP-6, symbol TLP185
- added C1, C5: 1µF, Capacitors_SMD:C_0805, symbol C_Small
- added C10, C12, C13, C3, C4, C6, C8: 100nF, Capacitors_SMD:C_0603, symbol C_Small
- added C11, C9: 1µF, Capacitors_SMD:C_0603, symbol C_Small
- added C2, C7: 470µF, Capacitors_ThroughHole:CP_Radial_D8.0mm_P2.50mm, symbol CP_Small
- added J1: limZ, Connect:bornier2, symbol Screw_Terminal_1x02
- added J10: COOLANT, Connect:bornier2, symbol Screw_Terminal_1x02
- added J11: SPINDLE, Connect:bornier3, symbol Screw_Terminal_1x03
- added J12: Z_CTRL, Connect:bornier3, symbol Screw_Terminal_1x03
- added J13: Z_ALIM, Connect:bornier2, symbol Screw_Terminal_1x02
- added J14: Y_CTRL, Connect:bornier3, symbol Screw_Terminal_1x03
- added J15: Y_ALIM, Connect:bornier2, symbol Screw_Terminal_1x02
- added J16: X_CTRL, Connect:bornier3, symbol Screw_Terminal_1x03
- added J17: X_ALIM, Connect:bornier2, symbol Screw_Terminal_1x02
- added J2: limY, Connect:bornier2, symbol Screw_Terminal_1x02
- added J3: limX, Connect:bornier2, symbol Screw_Terminal_1x02
- added J4: abort, Connect:bornier2, symbol Screw_Terminal_1x02
- added J5: stop, Connect:bornier2, symbol Screw_Terminal_1x02
- added J6: resume, Connect:bornier2, symbol Screw_Terminal_1x02
- added J7: probe, Connect:bornier2, symbol Screw_Terminal_1x02
- added J8: +12V, Connect:bornier2, symbol Screw_Terminal_1x02
- added J9: +24V, Connect:bornier2, symbol Screw_Terminal_1x02
- added P1, P4: CONN_01X08, Pin_Headers:Pin_Header_Straight_1x08_Pitch2.54mm, symbol CONN_01X08
- added P2: CONN_01X06, Pin_Headers:Pin_Header_Straight_1x06_Pitch2.54mm, symbol CONN_01X06
- added P3: CONN_01X10, Pin_Headers:Pin_Header_Straight_1x10_Pitch2.54mm, symbol CONN_01X10
- added P5: RESET, Pin_Headers:Pin_Header_Straight_1x02_Pitch2.54mm, symbol CONN_01X02
- added P6: RS232, Pin_Headers:Pin_Header_Straight_1x04_Pitch2.54mm, symbol CONN_01X04
- added R15: 10k, Resistors_SMD:R_0603, symbol R_Small
- added U10: 74HC125AN, SMD_Packages:SOIC-14_N, symbol 74HC125AN
- added U8: LM7805CT, Power_Integrations:TO-220, symbol LM7805CT
- added U9: 74HCT245P, SMD_Packages:SSOP-20, symbol 74HCT245P
- R1, R10, R11, R12, R13, R14, R2, R3, R4, R5, R6, R7, R8, R9: renamed from R?; footprint (none) -> Resistors_SMD:R_0603
Connections:
- net labels added: +24V, 3V3, 5V, AREF, IOREF, NC, RESET, RX, SCL, SDA, TX, VIN, b_out_COOLANT, b_out_DIR_X, b_out_DIR_Y, b_out_DIR_Z, b_out_ENABLE, b_out_SPINDLE_DIR, b_out_SPINDLE_PWM, b_out_STEP_X, b_out_STEP_Y, b_out_STEP_Z, in_ABORT, in_HOLD, in_LIMIT_X, in_LIMIT_Y, in_LIMIT_Z, in_PROBE, in_RESUME, out_COOLANT, out_DIR_X, out_DIR_Y, out_DIR_Z, out_ENABLE, out_SPINDLE_DIR, out_SPINDLE_PWM, out_STEP_X, out_STEP_Y, out_STEP_Z
- net labels removed: ABORT, LIMIT_X, LIMIT_Y, LIMIT_Z, PROBE, RESUME, STOP
- wire segments 37 -> 177
Other:
- moved on the sheet: R1, R10, R11, R12, R13, R14, R2, R3, R4, R5, R6, R7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

Commit message: Commit V1.0
Parts:
- removed P1, P4: CONN_01X08, Pin_Headers:Pin_Header_Straight_1x08_Pitch2.54mm, symbol CONN_01X08
- removed P2: CONN_01X06, Pin_Headers:Pin_Header_Straight_1x06_Pitch2.54mm, symbol CONN_01X06
- removed P3: CONN_01X10, Pin_Headers:Pin_Header_Straight_1x10_Pitch2.54mm, symbol CONN_01X10
- added J18: LED, Connect:bornier2, symbol Screw_Terminal_1x02
- added SHIELD1: ARDUINO_UNO_REV3_SHIELD, arduino_uno_rev3_shield:arduino_uno_rev3_grbl_shield, symbol ARDUINO_UNO_REV3_SHIELD
- added U1, U2, U3, U4, U5, U6, U7: TLP185, Opto-Devices:Toshiba_SOP_Pins1346_4.4x3.6mm_Pitch1.27mm, symbol TLP185
- J5: value stop -> hold
Connections:
- net labels added: +12V, RST, VCC
- net labels removed: 3V3, 5V, AREF, IOREF, NC, RESET, SCL, SDA, VIN
- wire segments 177 -> 185
- no-connect marks 0 -> 11
Other:
- moved on the sheet: C1, C11, C2, C5, C7, C9, J8, J9, U8
