File: arduino_uno_grbl_shield.kicad_pcb (KiCad board)
At the start: 2 copper layers, 122 x 56 mm, 65 parts, among them J1 limZ, J10 COOLANT, J11 SPINDLE, J12 Z_CTRL, J13 Z_ALIM, J14 Y_CTRL, J15 Y_ALIM, J16 X_CTRL, J17 X_ALIM, J18 LED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

Commit message: V1.1
Routing:
- net +5V: track 402.0 -> 403.7 mm
- net in_LIMIT_Y: track 103.7 -> 102.2 mm, vias 2 -> 1
Other:
- net class +24V: trace_width 2.8 -> 4; via_dia 2.8 -> 4
Changed lines of the file:
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@@
     (links 140)
     (no_connects 0)
-    (area 51.150001 61.3 192.157143 131.5)
+    (area 51.150001 61.3 192.5 132.5)
     (thickness 1.6)
     (drawings 77)
-    (tracks 388)
+    (tracks 389)
     (zones 0)
     (modules 65)
@@
     (35 F.Paste user hide)
     (36 B.SilkS user hide)
-    (37 F.SilkS user)
+    (37 F.SilkS user hide)
     (38 B.Mask user hide)
     (39 F.Mask user hide)
@@
     (pad_to_mask_clearance 0.2)
     (aux_axis_origin 64 126)
-    (visible_elements 7FFCEF9F)
+    (visible_elements 7FFCFF9F)
     (pcbplotparams
       (layerselection 0x3ffff_80000001)
@@
       (excludeedgelayer true)
       (linewidth 0.150000)
-      (plotframeref false)
-      (viasonmask false)
+      (plotframeref true)
+      (viasonmask true)
       (mode 1)
       (useauxorigin false)
@@
       (psnegative false)
       (psa4output false)
-      (plotreference true)
-      (plotvalue true)
+      (plotreference false)
+      (plotvalue false)
       (plotinvisibletext false)
       (padsonsilk false)
@@
   (net_class +24V ""
     (clearance 0.8)
-    (trace_width 2.8)
-    (via_dia 2.8)
+    (trace_width 4)
+    (via_dia 4)
     (via_drill 1)
     (uvia_dia 0.3)
@@
       (xy -0.113933 -2.757629) (xy -0.013056 -2.757714) (xy 0 -2.757714) (xy 0.10391 -2.757652)) (layer F.SilkS) (width 0.01))
   )
+  (target plus (at 60 130) (size 5) (width 0.15) (layer Edge.Cuts))
+  (target plus (at 190 130) (size 5) (width 0.15) (layer Edge.Cuts))
+  (target plus (at 190 65) (size 5) (width 0.15) (layer Edge.Cuts))
+  (target plus (at 60 65) (size 5) (width 0.15) (layer Edge.Cuts))
   (gr_text "GRBL SHIELD V1.0\n(c) 2017 Johann Delahayes" (at 104 122) (layer F.SilkS)
     (effects (font (size 1.5 1.5) (thickness 0.3)))
   )
-  (target plus (at 189 129) (size 5) (width 0.15) (layer Edge.Cuts))
-  (target plus (at 61 129) (size 5) (width 0.15) (layer Edge.Cuts))
-  (target plus (at 61 67) (size 5) (width 0.15) (layer Edge.Cuts))
-  (target plus (at 189 67) (size 5) (width 0.15) (layer Edge.Cuts))
   (dimension 48 (width 0.3) (layer Cmts.User)
     (gr_text "48,000 mm" (at 60.65 98 270) (layer Cmts.User)
@@
   (segment (start 140.714 112.141) (end 140.714 114.417) (width 0.3) (layer B.Cu) (net 2) (status 30))
   (segment (start 140.714 114.417) (end 140.704 114.427) (width 0.3) (layer B.Cu) (net 2) (status 30))
-  (segment (start 104.267 85.471) (end 104.267 80.772) (width 0.3) (layer B.Cu) (net 3))
+  (segment (start 104.267 85.471) (end 105.664 84.074) (width 0.3) (layer B.Cu) (net 3))
   (segment (start 130.046 112.522) (end 128.651 112.522) (width 0.3) (layer B.Cu) (net 3) (status 10))
   (segment (start 127.635 111.506) (end 128.651 112.522) (width 0.3) (layer B.Cu) (net 3))
@@
   (segment (start 99.568 90.17) (end 99.568 98.806) (width 0.3) (layer B.Cu) (net 3))
   (segment (start 104.267 85.471) (end 99.568 90.17) (width 0.3) (layer B.Cu) (net 3))
-  (segment (start 135.382 80.264) (end 135.382 73.66) (width 0.3) (layer B.Cu) (net 3) (status 20))
-  (via (at 135.382 80.264) (size 1.4) (drill 1) (layers F.Cu B.Cu) (net 3))
-  (segment (start 112.649 80.264) (end 135.382 80.264) (width 0.3) (layer F.Cu) (net 3))
-  (via (at 112.649 80.264) (size 1.4) (drill 1) (layers F.Cu B.Cu) (net 3))
-  (segment (start 104.775 80.264) (end 112.649 80.264) (width 0.3) (layer B.Cu) (net 3))
-  (segment (start 104.267 80.772) (end 104.775 80.264) (width 0.3) (layer B.Cu) (net 3))
+  (segment (start 135.382 76.073) (end 135.382 73.66) (width 0.3) (layer F.Cu) (net 3))
+  (segment (start 134.874 76.581) (end 135.382 76.073) (width 0.3) (layer F.Cu) (net 3))
+  (segment (start 106.807 76.581) (end 134.874 76.581) (width 0.3) (layer F.Cu) (net 3))
+  (segment (start 105.918 77.47) (end 106.807 76.581) (width 0.3) (layer F.Cu) (net 3))
+  (segment (start 105.918 83.82) (end 105.918 77.47) (width 0.3) (layer F.Cu) (net 3))
+  (segment (start 105.664 84.074) (end 105.918 83.82) (width 0.3) (layer F.Cu) (net 3))
+  (via (at 105.664 84.074) (size 1.4) (drill 1) (layers F.Cu B.Cu) (net 3))
   (segment (start 130.036 114.808) (end 130.036 116.84) (width 0.3) (layer B.Cu) (net 3) (status 30))
   (segment (start 130.046 112.522) (end 130.046 114.798) (width 0.3) (layer B.Cu) (net 3) (status 30))
@@
   (segment (start 82.284 114.808) (end 84.201 114.808) (width 0.3) (layer B.Cu) (net 4) (status 10))
   (segment (start 84.201 114.808) (end 85.864 114.808) (width 0.3) (layer B.Cu) (net 4) (status 20))
-  (segment (start 180.086 82.55) (end 180.086 107.696) (width 0.3) (layer F.Cu) (net 4))
+  (segment (start 182.086 84.55) (end 182.086 105.696) (width 0.3) (layer F.Cu) (net 4))
   (via (at 156.083 117.856) (size 1.4) (drill 1) (layers F.Cu B.Cu) (net 4))
   (segment (start 156.083 117.856) (end 154.305 116.078) (width 0.3) (layer F.Cu) (net 4))
   (segment (start 154.305 116.078) (end 154.305 109.855) (width 0.3) (layer F.Cu) (net 4))
   (segment (start 154.305 109.855) (end 155.956 108.204) (width 0.3) (layer F.Cu) (net 4))
-  (segment (start 180.086 82.55) (end 179.705 82.169) (width 0.3) (layer F.Cu) (net 4))
+  (segment (start 182.086 84.55) (end 179.705 82.169) (width 0.3) (layer F.Cu) (net 4))
   (segment (start 179.705 82.169) (end 173.482 82.169) (width 0.3) (layer F.Cu) (net 4))
   (segment (start 173.482 82.169) (end 171.958 82.169) (width 0.3) (layer F.Cu) (net 4))
@@
   (segment (start 179.578 108.204) (end 174.879 108.204) (width 0.3) (layer F.Cu) (net 4))
   (segment (start 174.879 108.204) (end 155.956 108.204) (width 0.3) (layer F.Cu) (net 4))
-  (segment (start 180.086 107.696) (end 179.578 108.204) (width 0.3) (layer F.Cu) (net 4))
+  (segment (start 182.086 105.696) (end 179.578 108.204) (width 0.3) (layer F.Cu) (net 4))
   (segment (start 137.414 84.201) (end 144.653 84.201) (width 0.3) (layer F.Cu) (net 4))
   (segment (start 145.669 85.217) (end 148.209 85.217) (width 0.3) (layer B.Cu) (net 4) (status 20))
@@
   (segment (start 172.466 106.68) (end 172.466 104.14) (width 0.3) (layer B.Cu) (net 16) (status 20))
   (segment (start 171.198 107.948) (end 172.466 106.68) (width 0.3) (layer B.Cu) (net 16))
-  (segment (start 79.375 97.536) (end 79.375 92.456) (width 2.8) (layer F.Cu) (net 17))
-  (segment (start 79.375 97.536) (end 81.534 99.695) (width 2.8) (layer F.Cu) (net 17))
-  (segment (start 124.714 99.695) (end 81.534 99.695) (width 2.8) (layer F.Cu) (net 17))
-  (segment (start 79.375 92.456) (end 74.422 87.503) (width 2.8) (layer F.Cu) (net 17))
-  (segment (start 151.13 94.996) (end 151.13 99.695) (width 2.8) (layer F.Cu) (net 17) (status 10))
+  (segment (start 79.375 97.536) (end 79.375 92.456) (width 4) (layer F.Cu) (net 17))
+  (segment (start 79.375 97.536) (end 81.534 99.695) (width 4) (layer F.Cu) (net 17))
+  (segment (start 124.714 99.695) (end 81.534 99.695) (width 4) (layer F.Cu) (net 17))
+  (segment (start 79.375 92.456) (end 74.422 87.503) (width 4) (layer F.Cu) (net 17))
+  (segment (start 151.13 94.996) (end 151.13 99.695) (width 4) (layer F.Cu) (net 17) (status 10))
   (segment (start 151.13 99.695) (end 152.273 99.695) (width 2.8) (layer F.Cu) (net 17))
-  (segment (start 124.714 94.996) (end 124.714 99.695) (width 2.8) (layer F.Cu) (net 17) (status 10))
-  (segment (start 177.546 97.917) (end 177.546 94.996) (width 2.8) (layer F.Cu) (net 17) (status 20))
-  (segment (start 175.768 99.695) (end 177.546 97.917) (width 2.8) (layer F.Cu) (net 17))
-  (segment (start 124.714 99.695) (end 152.273 99.695) (width 2.8) (layer F.Cu) (net 17))
-  (segment (start 152.273 99.695) (end 175.768 99.695) (width 2.8) (layer F.Cu) (net 17))
+  (segment (start 124.714 94.996) (end 124.714 99.695) (width 4) (layer F.Cu) (net 17) (status 10))
+  (segment (start 177.546 97.917) (end 177.546 94.996) (width 4) (layer F.Cu) (net 17) (status 20))
+  (segment (start 175.768 99.695) (end 177.546 97.917) (width 4) (layer F.Cu) (net 17))
+  (segment (start 124.714 99.695) (end 152.273 99.695) (width 4) (layer F.Cu) (net 17))
+  (segment (start 152.273 99.695) (end 175.768 99.695) (width 4) (layer F.Cu) (net 17))
   (segment (start 162.56 117.856) (end 162.56 118.872) (width 0.3) (layer B.Cu) (net 18) (status 10))
   (segment (start 161.798 107.823) (end 161.798 104.14) (width 0.3) (layer B.Cu) (net 18) (status 20))
